File: KiCad/Project/Schema_Experimento_Abordo.kicad_sch (KiCad schematic)
At the start: 29 parts, among them SW1 RESET, U1 ESP32-S3-WROOM-1, U2 BME280, U5 Micro_SD, U6 ZC323200, U7 SGP30, U9 AP2112K-3.3

Commit message: Esquematico limpio y probado. PCB Actualizado. Falta definir si se cambia el U9 por un Buck-boost
Parts:
- removed C1: 0.1uF, Capacitor_SMD:C_0805_2012Metric_Pad1.18x1.45mm_HandSolder, symbol Device:C
- removed C10, C11, C15, C4, C5, C7, C8: 100nF, Capacitor_SMD:C_0805_2012Metric_Pad1.18x1.45mm_HandSolder, symbol Device:C
- U2: footprint Package_LGA:Bosch_LGA-8_2.5x2.5mm_P0.65mm_ClockwisePinNumbering -> Connector_PinHeader_2.54mm:PinHeader_1x04_P2.54mm_Vertical
- U7: footprint SGP30:SGP30 -> Connector_PinHeader_2.54mm:PinHeader_1x04_P2.54mm_Vertical; symbol SGP30:SGP30 -> SGP30_Module:SGP30_Module; Availability Not in stock -> (none); Check_prices https://www.snapeda.com/parts/SGP30/Sensirion/view-part/?re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 -> (none); MF Sensirion AG -> (none); MP SGP30 -> (none); PROD_ID IC-14776 -> (none); Package None -> (none); Price None -> (none); SnapEDA_Link https://www.snapeda.com/parts/SGP30/Sensirion/view-part/?re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 -> (none)
- U8: footprint Package_TO_SOT_THT:TO-39-4 -> Connector_PinHeader_2.54mm:PinHeader_1x04_P2.54mm_Vertical
Connections:
- net D13 is gone; now on net CS MicroSD: U5.2 (CS)
- net D14 is gone; now on net RST LoRa: U4.6 (RESET)
- net D18 is gone; now on net SCK SPI: U4.4 (SCK), U5.4 (CLK)
- net D19 is gone; now on net MISO SPI: U4.2 (MISO), U5.5 (MISO)
- net D23 is gone; now on net MOSI SPI: U4.3 (MOSI), U5.3 (MOSI)
- net D26 is gone; now on net DIO0 LoRa: U4.11 (DIO0)
- net D27 is gone; now on net MPU6050 INT: U3.8 (INT)
- net D5 is gone; now on net NSS LoRa: U4.5 (NSS)
- net RX2 is gone; now on net GPS_RX: U6.2 (RX)
- net SCL I2C is gone; now on net SCL: R3.1, U1.25 (D32)
- net SDA I2C is gone; now on net SDA: R2.1, U1.24 (D33)
- net TX2 is gone; now on net GPS_TX: U6.3 (TX)
- net +3.3V: no longer U7.5 (VDDH)
- net GND: now also U1.40 (GND), U1.41 (GND), U3.7 (AD0), U6.SH1 (GND), U6.SH2 (GND), U6.SH3 (GND), U6.SH4 (GND); no longer U3. (AD0), U7.4 (R), U7.DIEPAD
- net D32 renamed SCL
- net SCL: now also U7.3 (SCL); no longer U7.6 (SCL)
- net D33 renamed SDA
- net SDA: now also U7.4 (SDA); no longer U7.3 (SDA)
Other:
- moved on the sheet: C2, U5
