File: KiCad/IGNIS-1/boards/rf/rf.kicad_pcb (KiCad board)
At the start: 2 copper layers, 62 x 62 mm, 11 parts, among them J30 SMA_antena, J42 Backplane_2x10, U30 RFM95W_SX1276_433MHz, U31 microSD

Commit message: 5 boards separados, falta ajustar dimensiones de BME280 y MQ-135
Parts:
- added J1: J_PWR_2x4, IGNIS1:J_PWR_2x4_Keyed, F.Cu at (119.4, 98.4)
- C30, C31: footprint Capacitor_SMD:C_0805_2012Metric -> Capacitor_THT:C_Disc_D7.5mm_W2.5mm_P5.00mm
- C32: footprint Capacitor_SMD:C_1210_3225Metric -> Capacitor_THT:CP_Radial_D8.0mm_P3.80mm
- moved C31 31.6 mm to (104.8, 82.5), turned to 0 degrees
- moved U31 28.8 mm to (108.6, 77.5), turned to -90 degrees
- moved C32 10.2 mm to (90.8, 80.6)
- moved C30 9.09 mm to (96.4, 86.4)
Connections:
- J42 pad 1: +3V3 -> unconnected-(J42-Pin_1-Pad1)
Routing:
- net +3V3: track 80.9 -> 0.65 mm
- net MISO: track 44.8 -> 0.00 mm
- net MOSI: track 46.3 -> 15.4 mm
- net SCK: track 109.8 -> 87.6 mm
- net CS_SD: track 56.5 -> 41.6 mm
- net GND: track 15.5 -> 3.23 mm, vias 41 -> 18

Commit message: Se agregaron tracks. PCB Cerebro libre de errores.
Routing:
- net GND: track 3.23 -> 132.8 mm
- net SCK: track 87.6 -> 160.1 mm, vias 0 -> 1
- net +3V3: track 0.65 -> 59.1 mm
- net MISO: track 0.00 -> 33.3 mm
- net CS_SD: track 41.6 -> 64.0 mm, vias 0 -> 1
- net MOSI: track 15.4 -> 37.7 mm

Commit message: Todos los boards pasan el check, tracks completos
Changed lines of the file:
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@@
 		(tags "CP Radial series Radial pin pitch 3.80mm diameter 8mm height 14mm Electrolytic Capacitor")
 		(property "Reference" "C32"
-			(at 1.9 -5.25 180)
+			(at 2.911 -5.25 180)
 			(layer "F.SilkS")
 			(effects
@@
 		(tags "C Disc series Radial pin pitch 5.00mm diameter 7.5mm width 2.5mm Capacitor")
 		(property "Reference" "C30"
-			(at 2.5 -2.5 180)
-			(layer "F.SilkS")
-			(effects
+			(at 2.46 0 180)
+			(layer "F.SilkS")
+			(effects
