File: KiCad/IGNIS-1/boards/rf/rf.kicad_sch (KiCad schematic)
At the start: 7 parts, among them J30 SMA_antena, J42 Backplane_2x10, U30 RFM95W_SX1276_433MHz, U31 microSD

Commit message: Tracks listos en PCB
Parts:
- removed C32: 100uF, Capacitor_SMD:C_1210_3225Metric, symbol Device:C
- added C32: 100uF, Capacitor_THT:CP_Radial_D5.0mm_P2.00mm, symbol Device:C_Polarized
- C30, C31: footprint Capacitor_SMD:C_0805_2012Metric -> Capacitor_SMD:C_0805_2012Metric_Pad1.18x1.45mm_HandSolder
Connections:
- net +3V3: now also C32.1
- net GND: now also C32.2
