File: KiCad/IGNIS-1/boards/rf/rf.kicad_sch (KiCad schematic)
At the start: 7 parts, among them J30 SMA_antena, J42 Backplane_2x10, U30 RFM95W_SX1276_433MHz, U31 microSD

Commit message: Energia: split en 2 boards (carga + energia) y redistribucion de rieles
- Board carga (5º): TP4056 + bateria + RBF + SW1 + TPS63020 -> +3V3 y VSW al bus
- Board energia (4º): MT3608 -> +5V al bus (toma VSW)
- Simbolos nuevos: TP4056, TPS63020; footprints TP4056_HW373, SW_Slide_SS12D00
- Bus: +3V3(p1), +5V(p19), VSW(p20), GND(2/4/11); backplane a header plano
- cerebro: quitada seccion de energia duplicada (U2/J1/J2/SW1/C1), +3V3 del bus
- sensores: quitado MT3608 (U3), +5V del bus alimenta MQ-135/GPS
- ZC323200 eliminado (sin uso)

Co-Authored-By: Claude Opus 4.8 <noreply@anthropic.com>
Parts:
- J42: footprint Connector_IDC:IDC-Header_2x10_P2.54mm_Vertical -> Connector_PinHeader_2.54mm:PinHeader_2x10_P2.54mm_Vertical
Changed lines of the file:
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@@
 			)
 		)
-		(property "Footprint" "Connector_IDC:IDC-Header_2x10_P2.54mm_Vertical"
+		(property "Footprint" "Connector_PinHeader_2.54mm:PinHeader_2x10_P2.54mm_Vertical"
 			(at 217.17 130.81 0)
 			(hide yes)
