File: KiCad/IGNIS-1/boards/rf/rf.kicad_sch (KiCad schematic)
At the start: 7 parts, among them J30 SMA_antena, J42 Backplane_2x10, U30 RFM95W_SX1276_433MHz, U31 microSD

Commit message: 5 boards separados, falta ajustar dimensiones de BME280 y MQ-135
Parts:
- added J1: J_PWR_2x4, IGNIS1:J_PWR_2x4_Keyed, symbol IGNIS1:J_PWR_2x4
Connections:
- net +3V3: now also J1.1 (+3V3); no longer J42.1 (Pin_1)
- no-connect marks 14 -> 15
Other:
- moved on the sheet: C30, C31, C32, J30, U30, U31
