File: KiCad/IGNIS-1/IGNIS-1.kicad_sch (KiCad schematic)
At the start: 0 parts

Commit message: Actualizado los boards de IGNIS - separado en 3 boards
Other:
- note added: "*** NO CANONICO / SOLO REFERENCIA *** Diseno real y fabricacion: boards/{cerebro,rf,sensores}. Este jerarquico NO refleja los cambios post-split (footprints HandSolder, caps polarizados THT, U1 eliminado). NO editar ni fabricar desde aqui."
Changed lines of the file:
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@@
 		(instances
 			(project "IGNIS-1"
-				(path "/58726030-ca17-4402-bd88-69b3f1ff686d" (page "2"))))
+				(path "/5d1facc0-7dac-40de-a8c6-d3ccfbbb88f2" (page "2"))))
 	)
 	(sheet
@@
 		(instances
 			(project "IGNIS-1"
-				(path "/58726030-ca17-4402-bd88-69b3f1ff686d" (page "3"))))
+				(path "/5d1facc0-7dac-40de-a8c6-d3ccfbbb88f2" (page "3"))))
 	)
 	(sheet
@@
 		(instances
 			(project "IGNIS-1"
-				(path "/58726030-ca17-4402-bd88-69b3f1ff686d" (page "4"))))
+				(path "/5d1facc0-7dac-40de-a8c6-d3ccfbbb88f2" (page "4"))))
 	)
 	(sheet
@@
 		(instances
 			(project "IGNIS-1"
-				(path "/58726030-ca17-4402-bd88-69b3f1ff686d" (page "5"))))
+				(path "/5d1facc0-7dac-40de-a8c6-d3ccfbbb88f2" (page "5"))))
 	)
 	(sheet
@@
 		(instances
 			(project "IGNIS-1"
-				(path "/58726030-ca17-4402-bd88-69b3f1ff686d" (page "6"))))
+				(path "/5d1facc0-7dac-40de-a8c6-d3ccfbbb88f2" (page "6"))))
+	)
+	(text "*** NO CANONICO / SOLO REFERENCIA ***\nDiseno real y fabricacion: boards/{cerebro,rf,sensores}.\nEste jerarquico NO refleja los cambios post-split\n(footprints HandSolder, caps polarizados THT, U1 eliminado).\nNO editar ni fabricar desde aqui."
+		(exclude_from_sim no)
+		(at 38.1 20.0 0)
+		(effects
+			(font (size 2.54 2.54) (bold yes))
+			(justify left bottom)
+		)
 	)
 	(sheet_instances
