File: KiCad/IGNIS-1/boards/cerebro/cerebro.kicad_pcb (KiCad board)
At the start: 2 copper layers, 62 x 62 mm, 22 parts, among them J1 LiPo_1S_in, J2 RBF_pin, J40 Backplane_2x10, Q1 MMBT3904, SW1 Main_SW, U10 ESP32-WROOM-32E DevKit 40p, U2 BuckBoost_3V3

Commit message: Update antes de mover a 4o board
Parts:
- BZ1: footprint Buzzer_Beeper:Buzzer_12x9.5RM7.6 -> IGNIS1:Buzzer_D12_P8.41
- C1: footprint Capacitor_SMD:C_0805_2012Metric_Pad1.18x1.45mm_HandSolder -> Capacitor_THT:CP_Radial_D6.3mm_P2.50mm
- C10, C2: footprint Capacitor_THT:CP_Radial_D5.0mm_P2.00mm -> Capacitor_THT:CP_Radial_D8.0mm_P3.80mm
- C11: footprint Capacitor_SMD:C_0805_2012Metric_Pad1.18x1.45mm_HandSolder -> Capacitor_THT:C_Disc_D7.5mm_W2.5mm_P5.00mm
- D4: footprint Diode_SMD:D_SOD-123 -> Diode_THT:D_DO-35_SOD27_P7.62mm_Horizontal
- J40: footprint Connector_PinHeader_2.54mm:PinHeader_2x10_P2.54mm_Vertical -> Connector_IDC:IDC-Header_2x10_P2.54mm_Vertical
- R10, R11, R12: footprint Resistor_SMD:R_0805_2012Metric_Pad1.20x1.40mm_HandSolder -> Resistor_THT:R_Axial_DIN0207_L6.3mm_D2.5mm_P7.62mm_Horizontal
- U2: value BuckBoost_3V3 -> TPS63020; footprint Connector_PinHeader_2.54mm:PinHeader_1x04_P2.54mm_Vertical -> IGNIS1:TPS63020_module
- moved U2 23.9 mm to (148.5, 93.4)
- moved D4 4.98 mm to (99.4, 123.8)
Connections:
- net /BUZZ_B renamed Net-(Q1-B)
- net /LEDP renamed Net-(D2-A)
- net /LEDS renamed Net-(D3-A)
- U10 pad 20: GND -> unconnected-(U10-5V-Pad20)
- U2 pad 2: GND -> +3V3
- U2 pad 3: /VSW -> GND
- U2 pad 4: +3V3 -> /VSW
