File: KiCad/IGNIS-1/boards/cerebro/cerebro.kicad_sch (KiCad schematic)
At the start: 18 parts, among them J1 LiPo_1S_in, J2 RBF_pin, J40 Backplane_2x10, Q1 MMBT3904, SW1 Main_SW, U10 ESP32-WROOM-32E DevKit 40p, U2 BuckBoost_3V3

Commit message: Update antes de mover a 4o board
Parts:
- BZ1: footprint Buzzer_Beeper:Buzzer_12x9.5RM7.6 -> IGNIS1:Buzzer_D12_P8.41
- C1: footprint Capacitor_SMD:C_0805_2012Metric_Pad1.18x1.45mm_HandSolder -> Capacitor_THT:CP_Radial_D6.3mm_P2.50mm
- C10, C2: footprint Capacitor_THT:CP_Radial_D5.0mm_P2.00mm -> Capacitor_THT:CP_Radial_D8.0mm_P3.80mm
- C11: footprint Capacitor_SMD:C_0805_2012Metric_Pad1.18x1.45mm_HandSolder -> Capacitor_THT:C_Disc_D7.5mm_W2.5mm_P5.00mm
- D2, D3: footprint LED_SMD:LED_0805_2012Metric_Pad1.15x1.40mm_HandSolder -> LED_THT:LED_D3.0mm
- D4: footprint Diode_SMD:D_SOD-123 -> Diode_THT:D_DO-35_SOD27_P7.62mm_Horizontal
- J40: footprint Connector_PinHeader_2.54mm:PinHeader_2x10_P2.54mm_Vertical -> Connector_IDC:IDC-Header_2x10_P2.54mm_Vertical
- Q1: footprint Package_TO_SOT_SMD:SOT-23 -> IGNIS1:Q_TO92_2N3904_EBC
- R10, R11, R12: footprint Resistor_SMD:R_0805_2012Metric_Pad1.20x1.40mm_HandSolder -> Resistor_THT:R_Axial_DIN0207_L6.3mm_D2.5mm_P7.62mm_Horizontal
- U2: value BuckBoost_3V3 -> TPS63020; footprint Connector_PinHeader_2.54mm:PinHeader_1x04_P2.54mm_Vertical -> IGNIS1:TPS63020_module; symbol IGNIS1:DCDC_Module -> IGNIS1:TPS63020
Connections:
- net +3V3: now also U2.2 (VOUT); no longer U2.4 (VOUT)
- net GND: now also U2.3 (GND), U2.5 (PS); no longer U10.20 (GND), U2.2 (GND)
- net VSW: now also U2.4 (EN); no longer U2.3 (EN)
- no-connect marks 17 -> 19
Other:
- moved on the sheet: C2
