File: KiCad/IGNIS-1/boards/cerebro/cerebro.kicad_sch (KiCad schematic)
At the start: 18 parts, among them J1 LiPo_1S_in, J2 RBF_pin, J40 Backplane_2x10, Q1 MMBT3904, SW1 Main_SW, U10 ESP32-WROOM-32E DevKit 40p, U2 TPS63020

Commit message: Energia: split en 2 boards (carga + energia) y redistribucion de rieles
- Board carga (5º): TP4056 + bateria + RBF + SW1 + TPS63020 -> +3V3 y VSW al bus
- Board energia (4º): MT3608 -> +5V al bus (toma VSW)
- Simbolos nuevos: TP4056, TPS63020; footprints TP4056_HW373, SW_Slide_SS12D00
- Bus: +3V3(p1), +5V(p19), VSW(p20), GND(2/4/11); backplane a header plano
- cerebro: quitada seccion de energia duplicada (U2/J1/J2/SW1/C1), +3V3 del bus
- sensores: quitado MT3608 (U3), +5V del bus alimenta MQ-135/GPS
- ZC323200 eliminado (sin uso)

Co-Authored-By: Claude Opus 4.8 <noreply@anthropic.com>
Parts:
- removed C1: 22uF, Capacitor_THT:CP_Radial_D6.3mm_P2.50mm, symbol Device:C
- removed J1: LiPo_1S_in, Connector_PinHeader_2.54mm:PinHeader_1x02_P2.54mm_Vertical, symbol Connector_Generic:Conn_01x02
- removed J2: RBF_pin, Connector_PinHeader_2.54mm:PinHeader_1x02_P2.54mm_Vertical, symbol Connector_Generic:Conn_01x02
- removed SW1: Main_SW, Connector_PinHeader_2.54mm:PinHeader_1x02_P2.54mm_Vertical, symbol Switch:SW_SPST
- removed U2: TPS63020, IGNIS1:TPS63020_module, symbol IGNIS1:TPS63020
- J40: footprint Connector_IDC:IDC-Header_2x10_P2.54mm_Vertical -> Connector_PinHeader_2.54mm:PinHeader_2x10_P2.54mm_Vertical
Connections:
- no-connect marks 19 -> 18
