File: KiCad/IGNIS-1/boards/cerebro/cerebro.kicad_sch (KiCad schematic)
At the start: 13 parts, among them J40 Backplane_2x10, Q1 MMBT3904, U10 ESP32-WROOM-32E DevKit 40p

Commit message: Iniciando cambio de pcb de cerebro
Parts:
- added J50: J_PWR_2x4, IGNIS1:J_PWR_2x4_Keyed, symbol IGNIS1:J_PWR_2x4
Connections:
- net +3V3: now also J50.1 (+3V3); no longer J40.1 (Pin_1)
- net CS_SD: no longer J40.15 (Pin_15)
- net DIO0: no longer J40.17 (Pin_17)
- net GND: now also J40.1 (Pin_1), J50.2 (GND), J50.4 (GND), J50.6 (GND), J50.8 (GND); no longer J40.11 (Pin_11), J40.2 (Pin_2), J40.4 (Pin_4)
- net GPS_RX: no longer J40.9 (Pin_9)
- net GPS_TX: no longer J40.8 (Pin_8)
- net LORA_RST: no longer J40.18 (Pin_18)
- net MISO: no longer J40.14 (Pin_14)
- net MOSI: no longer J40.13 (Pin_13)
- net MPU_INT: no longer J40.7 (Pin_7)
- net MQ_AOUT: no longer J40.10 (Pin_10)
- net NSS_LORA: no longer J40.16 (Pin_16)
- net SCK: no longer J40.12 (Pin_12)
- net SCL: no longer J40.6 (Pin_6)
- net SDA: now also J40.2 (Pin_2); no longer J40.5 (Pin_5)
- no-connect marks 18 -> 17
