File: KiCad/IGNIS-1/boards/cerebro/cerebro.kicad_sch (KiCad schematic)
At the start: 14 parts, among them J40 Backplane_2x10, J50 J_PWR_2x4, Q1 MMBT3904, U10 ESP32-WROOM-32E DevKit 40p

Commit message: 5 boards separados, falta ajustar dimensiones de BME280 y MQ-135
Parts:
- removed C2: 100uF, Capacitor_THT:CP_Radial_D8.0mm_P3.80mm, symbol Device:C_Polarized
- removed D2: PWR_grn, LED_THT:LED_D3.0mm, symbol Device:LED
- removed R10: 1k, Resistor_THT:R_Axial_DIN0207_L6.3mm_D2.5mm_P7.62mm_Horizontal, symbol Device:R
Connections:
- net +3V3: no longer J40.1 (Pin_1)
- no-connect marks 19 -> 21
Other:
- moved on the sheet: D3, J50, R11
