File: KiCad/IGNIS-1/boards/sensores/sensores.kicad_sch (KiCad schematic)
At the start: 12 parts, among them J41 Backplane_2x10, U20 BME280, U21 MPU6050, U22 MQ-135, U24 GPS NEO-6M, U3 Boost_5V

Commit message: Update antes de mover a 4o board
Parts:
- C20: footprint Capacitor_SMD:C_0805_2012Metric_Pad1.18x1.45mm_HandSolder -> Capacitor_THT:C_Disc_D7.5mm_W2.5mm_P5.00mm
- C4: footprint Capacitor_THT:CP_Radial_D6.3mm_P2.50mm -> Capacitor_THT:CP_Radial_D13.0mm_P5.00mm
- J41: footprint Connector_PinHeader_2.54mm:PinHeader_2x10_P2.54mm_Vertical -> Connector_IDC:IDC-Header_2x10_P2.54mm_Vertical
- R20, R21, R22, R23: footprint Resistor_SMD:R_0805_2012Metric_Pad1.20x1.40mm_HandSolder -> Resistor_THT:R_Axial_DIN0207_L6.3mm_D2.5mm_P7.62mm_Horizontal
- U21: footprint Connector_PinHeader_2.54mm:PinHeader_1x08_P2.54mm_Vertical -> IGNIS1:MPU6050_module
- U24: footprint ZC323200:XCVR_ZC323200 -> IGNIS1:GPS_NEO6M_module
- U3: footprint Connector_PinHeader_2.54mm:PinHeader_1x04_P2.54mm_Vertical -> IGNIS1:MT3608_module; symbol IGNIS1:DCDC_Module -> IGNIS1:Boost_MT3608
Connections:
- net +3V3: no longer U3.3 (EN)
- net +5V: now also U3.3 (OUT+); no longer U3.4 (VOUT)
- net GND: now also U3.4 (OUT-)
Other:
- moved on the sheet: C20, R20, R21, R22, R23, U22, U24
