File: KiCad/IGNIS-1/boards/sensores/sensores.kicad_pcb (KiCad board)
At the start: 2 copper layers, 62 x 62 mm, 16 parts, among them J1 J_PWR_2x4, J41 J_DAT, U20 BME280, U21 MPU6050, U22 MQ-135, U24 GPS NEO-6M

Commit message: Footprint BME280 propio + asignado (board sensores)
- Nuevo footprint IGNIS1:BME280_module (13.6x10.4mm, 4 THT P2.54
  VCC/GND/SCL/SDA, agujero montaje 3mm arriba-derecha).
- Asignado en simbolo maestro (default) y en instancia U20 del esquematico.
- PCB sensores: U20 cambia de PinHeader_1x04 generico a BME280_module;
  tracks viejos de U20 removidos (pads reubicados, falta rerutear).

Co-Authored-By: Claude Opus 4.8 <noreply@anthropic.com>
Parts:
- U20: footprint Connector_PinHeader_2.54mm:PinHeader_1x04_P2.54mm_Vertical -> IGNIS1:BME280_module
- moved U20 3.50 mm to (125.5, 104.9), turned to -90 degrees
Routing:
- net SCL: track 78.0 -> 73.0 mm
Changed lines of the file:
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@@
 		(embedded_fonts no)
 	)
-	(footprint "Connector_PinHeader_2.54mm:PinHeader_1x04_P2.54mm_Vertical"
-		(layer "F.Cu")
-		(at 123 102.5)
-		(descr "Through hole straight pin header, 1x04, 2.54mm pitch, single row")
-		(tags "Through hole pin header THT 1x04 2.54mm single row")
+	(footprint "IGNIS1:BME280_module"
+		(layer "F.Cu")
+		(at 125.5366 104.9152 -90)
+		(descr "BME280 breakout 13.6x10.4mm - 4 THT pins 1-row P2.54 on left (VCC/GND/SCL/SDA top->bottom), 1x 3mm mounting hole top-right. Module mounts face-up, pins down (mezzanine). Top view 1:1, no mirror. I2C 3.3V.")
 		(property "Reference" "U20"
-			(at 0 -2.38 0)
+			(at 0 -6.2 90)
 			(layer "F.SilkS")
 			(effects
@@
 		)
 		(property "Value" "BME280"
-			(at 0 10 0)
-			(layer "F.Fab")
-			(effects
-				(font
-					(size 1 1)
-					(thickness 0.15)
-				)
-			)
-		)
-		(property "Datasheet" "~"
-			(at 0 0 0)
+			(at 0 6.2 90)
+			(layer "F.Fab")
+			(effects
+				(font
+					(size 1 1)
+					(thickness 0.15)
+				)
+			)
+		)
+		(property "Datasheet" ""
+			(at 0 0 90)
 			(layer "F.Fab")
 			(hide yes)
@@
 		)
 		(property "Description" ""
-			(at 0 0 0)
+			(at 0 0 90)
 			(layer "F.Fab")
 			(hide yes)
@@
 		)
 		(property "KiLib_Generator" "connector/pin_header_socket"
-			(at 0 0 0)
+			(at 0 0 90)
 			(layer "F.SilkS")
 			(hide yes)
@@
 		(sheetname "/")
 		(sheetfile "sensores.kicad_sch")
-		(units
-			(unit
-				(name "A")
-				(pins "1" "2" "3" "4")
-			)
-		)
 		(attr through_hole)
 		(duplicate_pad_numbers_are_jumpers no)
-		(fp_line
-			(start -1.38 -1.38)
-			(end 0 -1.38)
+		(fp_rect
+			(start -6.8 -5.2)
+			(end 6.8 5.2)
 			(stroke
 				(width 0.12)
 				(type solid)
 			)
-			(layer "F.SilkS")
-		)
-		(fp_line
-			(start -1.38 0)
-			(end -1.38 -1.38)
-			(stroke
-				(width 0.12)
-				(type solid)
-			)
-			(layer "F.SilkS")
-		)
-		(fp_line
-			(start -1.38 1.27)
-			(end -1.38 9)
-			(stroke
-				(width 0.12)
-				(type solid)
-			)
-			(layer "F.SilkS")
-		)
-		(fp_line
-			(start -1.38 1.27)
-			(end 1.38 1.27)
-			(stroke
-				(width 0.12)
-				(type solid)
-			)
-			(layer "F.SilkS")
-		)
-		(fp_line
-			(start -1.38 9)
-			(end 1.38 9)
-			(stroke
-				(width 0.12)
-				(type solid)
-			)
-			(layer "F.SilkS")
-		)
-		(fp_line
-			(start 1.38 1.27)
-			(end 1.38 9)
-			(stroke
-				(width 0.12)
-				(type solid)
-			)
+			(fill no)
 			(layer "F.SilkS")
 		)
 		(fp_rect
-			(start -1.77 -1.77)
-			(end 1.77 9.39)
+			(start -7.05 -5.45)
+			(end 7.05 5.45)
 			(stroke
 				(width 0.05)
@@
 			(layer "F.CrtYd")
 		)
-		(fp_line
-			(start -1.27 -0.635)
-			(end -0.635 -1.27)
-			(stroke
-				(width 0.1)
-				(type solid)
-			)
-			(layer "F.Fab")
-		)
-		(fp_line
-			(start -1.27 8.89)
-			(end -1.27 -0.635)
-			(stroke
-				(width 0.1)
-				(type solid)
-			)
-			(layer "F.Fab")
-		)
-		(fp_line
-			(start -0.635 -1.27)
-			(end 1.27 -1.27)
-			(stroke
-				(width 0.1)
-				(type solid)
-			)
-			(layer "F.Fab")
-		)
-		(fp_line
-			(start 1.27 -1.27)
-			(end 1.27 8.89)
-			(stroke
-				(width 0.1)
-				(type solid)
-			)
-			(layer "F.Fab")
-		)
-		(fp_line
-			(start 1.27 8.89)
-			(end -1.27 8.89)
-			(stroke
-				(width 0.1)
-				(type solid)
-			)
-			(layer "F.Fab")
-		)
-		(fp_text user "${REFERENCE}"
-			(at 0 3.81 90)
-			(layer "F.Fab")
-			(effects
-				(font
-					(size 1 1)
-					(thickness 0.15)
-				)
-			)
+		(fp_text user "SDA"
+			(at -2.8 3.81 90)
+			(layer "F.SilkS")
+			(effects
+				(font
+					(size 0.9 0.9)
+					(thickness 0.15)
+				)
+				(justify right)
+			)
+		)
+		(fp_text user "SCL"
+			(at -2.8 1.27 90)
+			(layer "F.SilkS")
+			(effects
+				(font
+					(size 0.9 0.9)
+					(thickness 0.15)
+				)
+				(justify right)
+			)
+		)
+		(fp_text user "GND"
+			(at -2.8 -1.27 90)
+			(layer "F.SilkS")
+			(effects
+				(font
+					(size 0.9 0.9)
+					(thickness 0.15)
+				)
+				(justify right)
+			)
+		)
+		(fp_text user "VCC"
+			(at -2.8 -3.81 90)
+			(layer "F.SilkS")
+			(effects
+				(font
+					(size 0.9 0.9)
+					(thickness 0.15)
+				)
+				(justify right)
+			)
+		)
+		(pad "" np_thru_hole circle
+			(at 4 -2.2 270)
+			(size 3 3)
+			(drill 3)
+			(layers "*.Cu" "*.Mask")
 		)
 		(pad "1" thru_hole rect
-			(at 0 0)
-			(size 1.7 1.7)
+			(at -5.08 -3.81 270)
+			(size 1.8 1.8)
 			(drill 1)
 			(layers "*.Cu" "*.Mask")
@@
 		)
 		(pad "2" thru_hole circle
-			(at 0 2.54)
-			(size 1.7 1.7)
+			(at -5.08 -1.27 270)
+			(size 1.8 1.8)
 			(drill 1)
 			(layers "*.Cu" "*.Mask")
@@
 		)
 		(pad "3" thru_hole circle
-			(at 0 5.08)
-			(size 1.7 1.7)
+			(at -5.08 1.27 270)
+			(size 1.8 1.8)
 			(drill 1)
 			(layers "*.Cu" "*.Mask")
@@
 		)
 		(pad "4" thru_hole circle
-			(at 0 7.62)
-			(size 1.7 1.7)
+			(at -5.08 3.81 270)
+			(size 1.8 1.8)
 			(drill 1)
 			(layers "*.Cu" "*.Mask")
@@
 		)
 		(embedded_fonts no)
-		(model "${KICAD10_3DMODEL_DIR}/Connector_PinHeader_2.54mm.3dshapes/PinHeader_1x04_P2.54mm_Vertical.step"
-			(offset
-				(xyz 0 0 0)
-			)
-			(scale
-				(xyz 1 1 1)
-			)
-			(rotate
-				(xyz 0 0 0)
-			)
-		)
 	)
 	(footprint "Capacitor_THT:C_Disc_D7.5mm_W2.5mm_P5.00mm"
@@
 	(segment
 		(start 123 107.58)
-		(end 118.910825 103.490825)
-		(width 0.25)
-		(layer "B.Cu")
-		(net "SCL")
-	)
-	(segment
-		(start 114.094175 101.765825)
-		(end 118.910825 101.765825)
-		(width 0.25)
-		(layer "B.Cu")
-		(net "SCL")
-	)
-	(segment
-		(start 118.910825 103.490825)
-		(end 118.910825 101.765825)
+		(end 122.0927 106.6727)
 		(width 0.25)
 		(layer "B.Cu")
@@
 	(segment
 		(start 100.98 114.88)
-		(end 114.094175 101.765825)
+		(end 109.1873 106.6727)
 		(width 0.25)
 		(layer "B.Cu")
+		(net "SCL")
+	)
+	(segment
+		(start 122.0927 106.6727)
+		(end 109.1873 106.6727)
+		(width 0.25)
+		(layer "B.Cu")
