File: KiCad/IGNIS-1/sheets/sensors.kicad_sch (KiCad schematic)
At the start: 11 parts, among them U20 BME280, U21 MPU6050, U22 MQ-135, U24 GPS NEO-6M, U3 Boost_5V

Commit message: Update antes de mover a 4o board
Parts:
- U3: symbol IGNIS1:DCDC_Module -> IGNIS1:Boost_MT3608
Connections:
- net +3V3: no longer U3.3 (EN)
- net +5V: now also U3.3 (OUT+); no longer U3.4 (VOUT)
- net GND: now also U3.4 (OUT-)
Changed lines of the file:
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@@
 	)
 	(symbol
-		(lib_id "IGNIS1:DCDC_Module")
+		(lib_id "IGNIS1:Boost_MT3608")
 		(at 95.25 109.22 0)
 		(unit 1)
@@
 	)
 	(symbol
-		(lib_id "power:+3V3")
-		(at 87.63 109.22 0)
-		(unit 1)
-		(exclude_from_sim no)
-		(in_bom yes)
-		(on_board yes)
-		(dnp no)
-		(property "Reference" "#PWR_S16" (at 87.63 100.33 0) (effects (font (size 1.27 1.27))))
-		(property "Value" "+3V3" (at 87.63 118.11 0) (effects (font (size 1.27 1.27))))
-		(property "Footprint" "" (at 87.63 109.22 0) (effects (font (size 1.27 1.27)) (hide yes)))
-		(property "Datasheet" "~" (at 87.63 109.22 0) (effects (font (size 1.27 1.27)) (hide yes)))
-		(pin "1")
-		(instances
+		(lib_id "power:GND")
+		(at 102.87 111.76 0)
+		(unit 1)
+		(exclude_from_sim no)
+		(in_bom yes)
+		(on_board yes)
+		(dnp no)
+		(property "Reference" "#PWR_S16" (at 102.87 102.87 0) (effects (font (size 1.27 1.27))))
+		(property "Value" "GND" (at 102.87 120.65 0) (effects (font (size 1.27 1.27))))
+		(property "Footprint" "" (at 102.87 111.76 0) (effects (font (size 1.27 1.27)) (hide yes)))
+		(property "Datasheet" "~" (at 102.87 111.76 0) (effects (font (size 1.27 1.27)) (hide yes)))
+		(pin "1")
+		(instances
