File: KiCad/IGNIS-1/sheets/sensors.kicad_sch (KiCad schematic)
At the start: 11 parts, among them U20 BME280, U21 MPU6050, U22 MQ-135, U24 GPS NEO-6M, U3 Boost_5V

Commit message: Footprint BME280 propio + asignado (board sensores)
- Nuevo footprint IGNIS1:BME280_module (13.6x10.4mm, 4 THT P2.54
  VCC/GND/SCL/SDA, agujero montaje 3mm arriba-derecha).
- Asignado en simbolo maestro (default) y en instancia U20 del esquematico.
- PCB sensores: U20 cambia de PinHeader_1x04 generico a BME280_module;
  tracks viejos de U20 removidos (pads reubicados, falta rerutear).

Co-Authored-By: Claude Opus 4.8 <noreply@anthropic.com>
Parts:
- U20: footprint Connector_PinHeader_2.54mm:PinHeader_1x04_P2.54mm_Vertical -> IGNIS1:BME280_module
Changed lines of the file:
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@@
 		(property "Reference" "U20" (at 50.8 62.230000000000004 0) (effects (font (size 1.27 1.27))))
 		(property "Value" "BME280" (at 50.8 80.01 0) (effects (font (size 1.27 1.27))))
-		(property "Footprint" "Connector_PinHeader_2.54mm:PinHeader_1x04_P2.54mm_Vertical" (at 50.8 71.12 0) (effects (font (size 1.27 1.27)) (hide yes)))
+		(property "Footprint" "IGNIS1:BME280_module" (at 50.8 71.12 0) (effects (font (size 1.27 1.27)) (hide yes)))
 		(property "Datasheet" "~" (at 50.8 71.12 0) (effects (font (size 1.27 1.27)) (hide yes)))
 		(pin "1")
