File: KiCad/IGNIS-1/boards/energia/energia.kicad_sch (KiCad schematic)
At the start: 6 parts, among them J40 Backplane, U3 Boost_5V

Commit message: 5 boards separados, falta ajustar dimensiones de BME280 y MQ-135
Parts:
- removed J40: Backplane, Connector_PinHeader_2.54mm:PinHeader_2x10_P2.54mm_Vertical, symbol Connector_Generic:Conn_02x10_Odd_Even
- added C1: 22uF, Capacitor_THT:CP_Radial_D6.3mm_P2.50mm, symbol Device:C
- added C2: 100uF, Capacitor_THT:CP_Radial_D8.0mm_P3.80mm, symbol Device:C
- added J1: J_PWR_2x4, IGNIS1:J_PWR_2x4_Keyed, symbol IGNIS1:J_PWR_2x4
- added U2: TPS63020, IGNIS1:TPS63020_module, symbol IGNIS1:TPS63020
Connections:
- net +3V3: now also C2.1, J1.1 (+3V3), U2.2 (VOUT)
- net +5V: now also J1.3 (+5V)
- net GND: now also C1.2, C2.2, J1.2 (GND), J1.4 (GND), J1.6 (GND), J1.8 (GND), U2.3 (GND), U2.5 (PS)
- net VSW: now also C1.1, J1.5 (VSW), U2.1 (VIN), U2.4 (EN)
- no-connect marks 15 -> 1
Other:
- moved on the sheet: D2, R10
