File: KiCad/IGNIS-1/placa_poder_cerebro/placa_poder_cerebro.kicad_pcb (KiCad board)
At the start: 2 copper layers, 58 x 100 mm, 26 parts, among them J30 SMA_antena, J50 Conn_02x06_Odd_Even, Q1 MMBT3904, U10 ESP32-WROOM-32E DevKit 40p, U2 TPS63020, U30 RFM95W_SX1276_433MHz, U31 microSD

Commit message: Rutear placa_poder_cerebro y reposicionar footprints de placa_sensores
Co-Authored-By: Claude Opus 4.8 <noreply@anthropic.com>
Parts:
- C30, C31: moved to B.Cu
- moved D3 66.2 mm to (104.0, 64.5), turned to -90 degrees
- moved C32 63.4 mm to (105.5, 137.5), turned to -90 degrees
- moved C30 56.5 mm to (119.5, 137.9), turned to -90 degrees
- moved C2 50.8 mm to (129.0, 126.5), turned to 180 degrees
- moved C11 48.8 mm to (140.0, 55.0), turned to 90 degrees
- moved R11 38.8 mm to (104.0, 71.9), turned to 90 degrees
- moved C10 37.6 mm to (146.0, 55.0), turned to 90 degrees
- moved C31 32.5 mm to (141.4, 67.0)
- moved R12 31.3 mm to (125.5, 111.1), turned to -90 degrees
- moved R10 21.1 mm to (128.6, 111.6), turned to 180 degrees
- moved C5 16.6 mm to (139.0, 94.5), turned to 180 degrees
- moved C1 7.93 mm to (139.0, 99.5), turned to 180 degrees
- moved D4 7.83 mm to (105.0, 114.0), turned to 0 degrees
- moved J50 2.54 mm to (107.5, 120.0)
- moved D2 1.16 mm to (130.0, 117.0)
Routing:
- net GND: track 0.00 -> 326.6 mm, vias 0 -> 16
- net +3V3: track 0.00 -> 207.6 mm, vias 0 -> 15
- net MOSI: track 0.00 -> 188.8 mm, vias 0 -> 9
- net MISO: track 0.00 -> 175.4 mm, vias 0 -> 4
- net SCK: track 0.00 -> 166.7 mm, vias 0 -> 6
- net NSS_LORA: track 0.00 -> 96.0 mm, vias 0 -> 1
- net GPS_TX: track 0.00 -> 87.0 mm
- net LORA_RST: track 0.00 -> 86.9 mm
- net DIO0: track 0.00 -> 83.7 mm
- net SCL: track 0.00 -> 79.4 mm
- net VSW: track 0.00 -> 77.3 mm, vias 0 -> 3
- net MPU_INT: track 0.00 -> 70.6 mm, vias 0 -> 2
- net SDA: track 0.00 -> 62.2 mm
- net GPS_RX: track 0.00 -> 61.6 mm, vias 0 -> 2
- net MQ_AOUT: track 0.00 -> 58.6 mm, vias 0 -> 2
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- added copper zone on B.Cu, net GND
