File: KiCad/IGNIS-1/placa_sensores/placa_sensores.kicad_pcb (KiCad board)
At the start: 2 copper layers, 58 x 100 mm, 21 parts, among them J1 LiPo_1S, J2 RBF_pin, J50 Conn_02x06_Odd_Even, SW1 Main_SW, U20 BME280, U21 MPU6050, U22 MQ-135, U24 GPS NEO-6M, U3 Boost_5V, U40 TP4056

Commit message: Rutear placa_poder_cerebro y reposicionar footprints de placa_sensores
Co-Authored-By: Claude Opus 4.8 <noreply@anthropic.com>
Parts:
- J50: moved to B.Cu
- moved J50 45.5 mm to (150.5, 120.0), turned to 180 degrees
- moved J1 43.7 mm to (105.7, 116.1)
- moved SW1 43.7 mm to (104.5, 136.7)
- moved J2 43.5 mm to (104.7, 124.8)
- moved R20 7.00 mm to (113.0, 125.9), turned to -90 degrees
- moved R22 6.71 mm to (144.2, 135.7)
- moved R23 6.71 mm to (144.2, 124.3)
- moved C20 6.71 mm to (135.7, 124.3)
- moved U20 6.37 mm to (123.0, 123.5)
- moved R21 5.30 mm to (117.8, 115.4)
Routing:
- net VSW: track 59.7 -> 0.00 mm
- net VBAT_P: track 40.4 -> 0.00 mm
- net BATT: track 31.2 -> 0.00 mm
- net GND: track 8.53 -> 34.6 mm, vias 0 -> 1
- net MQ_AOUT: track 43.1 -> 18.2 mm, vias 1 -> 0
- net Net-(U22-A0): track 0.00 -> 17.6 mm, vias 0 -> 1
- net SDA: track 16.7 -> 7.22 mm
- net +5V: track 0.00 -> 8.72 mm, vias 0 -> 1
- net SCL: track 8.71 -> 0.00 mm
- net VRBF: track 6.89 -> 0.00 mm
- net +3V3: track 11.2 -> 9.18 mm, vias 0 -> 1
